Commit message: add aruco gazebo model

File: src/m2wr_description/urdf/m2wr.xacro (robot description, xacro)
@@ -15,5 +15,6 @@
     <collision name="collision_chassis">
       <geometry>
-        <box size="0.5 0.3 0.07"/>
+        <!--box size="0.3 0.3 0.07"/-->
+        <mesh filename="package://m2wr_description/meshes/arucox0.dae"/>
       </geometry>
     </collision>
@@ -21,11 +22,12 @@
       <origin rpy="0 0 0" xyz="0 0 0"/>
       <geometry>
-        <box size="0.5 0.3 0.07"/>
+        <!--box size="0.3 0.3 0.07"/-->
+        <mesh filename="package://m2wr_description/meshes/arucox0.dae"/>
       </geometry>
-      <material name="blue"/>
+      <!--material name="blue"/-->
     </visual>
     <!-- caster front -->
     <collision name="caster_front_collision">
-      <origin rpy=" 0 0 0" xyz="0.35 0 -0.05"/>
+      <origin rpy=" 0 0 0" xyz="0.25 0 -0.05"/>
       <geometry>
         <sphere radius="0.05"/>
@@ -43,5 +45,5 @@
     </collision>
     <visual name="caster_front_visual">
-      <origin rpy=" 0 0 0" xyz="0.2 0 -0.05"/>
+      <origin rpy=" 0 0 0" xyz="0.15 0 -0.05"/>
       <geometry>
         <sphere radius="0.05"/>
@@ -50,6 +52,6 @@
   </link>
   <xacro:link_wheel name="link_right_wheel"/>
-  <xacro:joint_wheel name="joint_right_wheel" child="link_right_wheel" origin_xyz="-0.05 0.15 0"/>
+  <xacro:joint_wheel name="joint_right_wheel" child="link_right_wheel" origin_xyz="-0.05 0.2 0"/>
   <xacro:link_wheel name="link_left_wheel"/>
-  <xacro:joint_wheel name="joint_left_wheel" child="link_left_wheel" origin_xyz="-0.05 -0.15 0"/>
+  <xacro:joint_wheel name="joint_left_wheel" child="link_left_wheel" origin_xyz="-0.05 -0.2 0"/>
 </robot>
